Commit message: removing old models and worlds, adding in ported urdf files

File: cvg_sim_gazebo/urdf/quadrotor.urdf.xacro (robot description, xacro)
@@ -1,11 +1,130 @@
 <?xml version="1.0"?>
-<robot name="quadrotor"
-    xmlns:sensor="http://playerstage.sourceforge.net/gazebo/xmlschema/#sensor"
-    xmlns:controller="http://playerstage.sourceforge.net/gazebo/xmlschema/#controller"
-    xmlns:interface="http://playerstage.sourceforge.net/gazebo/xmlschema/#interface"
-    xmlns:xacro="http://playerstage.sourceforge.net/gazebo/xmlschema/#interface">
-    <!-- Included URDF Files -->
-    <include filename="$(find cvg_sim_gazebo)/urdf/quadrotor_base.urdf.xacro" />
-    <!-- Instantiate quadrotor_base_macro once (has no parameters atm) -->
-    <quadrotor_base_macro />
+<robot name="quadrotor" xmlns:xacro="http://www.ros.org/wiki/xacro">
+	<!-- Include URDF Files -->
+	<xacro:include filename="$(find cvg_sim_gazebo)/urdf/sensors/generic_camera.urdf.xacro" />
+	<xacro:include filename="$(find cvg_sim_gazebo)/urdf/sensors/sonar_sensor.urdf.xacro" />
+	<!-- End Include URDF Files -->
+	<!-- The body of the quadrotor -->
+	<link name="base_link">
+		<inertial>
+			<mass value="1.477" />
+			<origin xyz="0 0 0" />
+			<inertia ixx="0.01152" ixy="0.0" ixz="0.0" iyy="0.01152" iyz="0.0" izz="0.0218" />
+		</inertial>
+		<visual>
+			<origin xyz="0 0 0" rpy="0 0 0" />
+			<geometry>
+				<mesh filename="model://quadrotor/meshes/quadrotor_4.dae"/>
+			</geometry>
+		</visual>
+		<collision>
+			<origin xyz="0 0 0" rpy="0 0 0" />
+			<geometry>
+				<mesh filename="model://quadrotor/meshes/quadrotor_4.stl"/>
+			</geometry>
+		</collision>
+	</link>
+	<!-- Forward facing camera -->
+	<xacro:generic_camera name="front" sim_name="ardrone" parent="base_link" update_rate="60" res_x="640" res_y="360" image_format="R8G8B8" hfov="${81*M_PI/180}">
+		<origin xyz="0.21 0.0 0.01" rpy="0 0 0"/>
+	</xacro:generic_camera>
+	<!-- Downward facing camera -->
+	<xacro:generic_camera name="bottom" sim_name="ardrone" parent="base_link" update_rate="60" res_x="640" res_y="360" image_format="R8G8B8" hfov="${81*M_PI/180}">
+		<origin xyz="0.15 0.0 0.0" rpy="0 -${M_PI/2} 0"/>
+	</xacro:generic_camera>
+	<!-- Sonar height sensor -->
+	<xacro:sonar_sensor name="sonar" parent="base_link" ros_topic="sonar_height" update_rate="10" min_range="0.01" max_range="3.0" field_of_view="${40*M_PI/180}" ray_count="3">
+		<origin xyz="-0.15 0.0 0.0" rpy="0 ${90*M_PI/180} 0"/>
+	</xacro:sonar_sensor>
+	<!-- Gazebo Controller Plugins -->
+	<gazebo>
+		<static>false</static>
+			<!-- Gazebo Controller Plugins -->
+      <plugin name="quadrotor_simple_controller" filename="libhector_gazebo_quadrotor_simple_controller.so">
+        <alwaysOn>true</alwaysOn>
+        <updateRate>0.0</updateRate>
+        <bodyName>base_link</bodyName>
+        <stateTopic>ground_truth/state</stateTopic>
+        <imuTopic>ardrone/imu</imuTopic>
+        <topicName>cmd_vel</topicName>
+        <rollpitchProportionalGain>10.0</rollpitchProportionalGain>
+        <rollpitchDifferentialGain>5.0</rollpitchDifferentialGain>
+        <rollpitchLimit>0.5</rollpitchLimit>
+        <yawProportionalGain>2.0</yawProportionalGain>
+        <yawDifferentialGain>1.0</yawDifferentialGain>
+        <yawLimit>1.5</yawLimit>
+        <velocityXYProportionalGain>5.0</velocityXYProportionalGain>
+        <velocityXYDifferentialGain>1.0</velocityXYDifferentialGain>
+        <velocityXYLimit>2</velocityXYLimit>
+        <velocityZProportionalGain>5.0</velocityZProportionalGain>
+        <velocityZDifferentialGain>1.0</velocityZDifferentialGain>
+        <velocityZLimit>0.5</velocityZLimit>
+        <maxForce>30</maxForce>
+        <motionSmallNoise>0.05</motionSmallNoise>
+        <motionDriftNoise>0.03</motionDriftNoise>
+        <motionDriftNoiseTime>5.0</motionDriftNoiseTime>
+      </plugin>
+      <plugin name="quadrotor_state_controller" filename="libhector_gazebo_quadrotor_state_controller.so">
+        <alwaysOn>true</alwaysOn>
+        <updateRate>0.0</updateRate>
+        <bodyName>base_link</bodyName>
+        <stateTopic>ground_truth/state</stateTopic>
+        <imuTopic>ardrone/imu</imuTopic>
+        <sonarTopic>sonar_height</sonarTopic>
+        <topicName>cmd_vel</topicName>
+      </plugin>
+			<plugin name="quadrotor_imu_sim" filename="libhector_gazebo_ros_imu.so">
+				<alwaysOn>true</alwaysOn>
+				<updateRate>100.0</updateRate>
+				<bodyName>base_link</bodyName>
+				<frameId>ardrone_base_link</frameId>
+				<topicName>/ardrone/imu</topicName>
+				<rpyOffsets>0 0 0</rpyOffsets> <!-- deprecated -->
+				<gaussianNoise>0</gaussianNoise>  <!-- deprecated -->
+				<accelDrift>0.5 0.5 0.5</accelDrift>
+				<accelGaussianNoise>0.35 0.35 0.3</accelGaussianNoise>
+				<rateDrift>0.0 0.0 0.0</rateDrift>
+				<rateGaussianNoise>0.00 0.00 0.00</rateGaussianNoise>
+				<headingDrift>0.0</headingDrift>
+				<headingGaussianNoise>0.00</headingGaussianNoise>
+			</plugin>
+			<plugin name="quadrotor_baro_sim" filename="libhector_gazebo_ros_baro.so">
+				<alwaysOn>true</alwaysOn>
+				<updateRate>10.0</updateRate>
+				<bodyName>base_link</bodyName>
+				<topicName>pressure_height</topicName>
+				<altimeterTopicName>altimeter</altimeterTopicName>
+				<offset>0</offset>
+				<drift>0.1</drift>
+				<gaussianNoise>0.5</gaussianNoise>
+			</plugin>
+			<plugin name="quadrotor_magnetic_sim" filename="libhector_gazebo_ros_magnetic.so">
+				<alwaysOn>true</alwaysOn>
+				<updateRate>10.0</updateRate>
+				<bodyName>base_link</bodyName>
+				<topicName>magnetic</topicName>
+				<offset>0 0 0</offset>
+				<drift>0.0 0.0 0.0</drift>
+				<gaussianNoise>1.3e-2 1.3e-2 1.3e-2</gaussianNoise>
+			</plugin>
+			<plugin name="quadrotor_gps_sim" filename="libhector_gazebo_ros_gps.so">
+				<alwaysOn>true</alwaysOn>
+				<updateRate>4.0</updateRate>
+				<bodyName>base_link</bodyName>
+				<topicName>fix</topicName>
+				<velocityTopicName>fix_velocity</velocityTopicName>
+				<drift>5.0 5.0 5.0</drift>
+				<gaussianNoise>0.1 0.1 0.1</gaussianNoise>
+				<velocityDrift>0 0 0</velocityDrift>
+				<velocityGaussianNoise>0.1 0.1 0.1</velocityGaussianNoise>
+			</plugin>
+			<plugin name="quadrotor_groundtruth_sim" filename="libgazebo_ros_p3d.so">
+				<alwaysOn>true</alwaysOn>
+				<updateRate>100.0</updateRate>
+				<bodyName>base_link</bodyName>
+				<topicName>ground_truth/state</topicName>
+				<gaussianNoise>0.0</gaussianNoise>
+				<frameName>map</frameName>
+			</plugin>
+	</gazebo>
 </robot>

File: cvg_sim_gazebo/urdf/sensors/generic_camera.urdf.xacro (robot description, xacro)
@@ -1,90 +1,53 @@
 <?xml version="1.0"?>
-<robot xmlns:sensor="http://playerstage.sourceforge.net/gazebo/xmlschema/#sensor"
-xmlns:controller="http://playerstage.sourceforge.net/gazebo/xmlschema/#controller"
-xmlns:interface="http://playerstage.sourceforge.net/gazebo/xmlschema/#interface"
-  xmlns:xacro="http://ros.org/wiki/xacro"
-  >
-    <property name="M_PI" value="3.1415926535897931" />
-    <xacro:macro name="generic_camera" params="name sim_name parent *origin update_rate res_x res_y image_format hfov">
-      <joint name="${name}_joint" type="fixed">
-        <insert_block name="origin" />
-        <parent link="${parent}"/>
-        <child link="${name}_link"/>
-      </joint>
-      <link name="${name}_link">
-        <inertial>
-          <mass value="0.001" />
-          <origin xyz="0 0 0" rpy="0 0 0" />
-          <inertia ixx="0.0001" ixy="0" ixz="0" iyy="0.0001" iyz="0" izz="0.0001" />
-        </inertial>
-        <visual>
-          <origin xyz="0 0 0" rpy="0 0 0" />
-          <geometry>
-            <box size="0.01 0.01 0.01" />
-          </geometry>
-	  <material name="Blue">
-      <color rgba="0.0 0.0 0.8 1"/>
-    </material>
-        </visual>
-        <collision>
-          <origin xyz="0 0 0" rpy="0 0 0" />
-          <geometry>
-            <box size="0.01 0.01 0.01" />
-          </geometry>
-        </collision>
-      </link>
-    <joint name="${name}_optical_joint" type="fixed">
-      <origin xyz="0 0 0" rpy="${-M_PI/2} 0.0 ${-M_PI/2}" />
-      <parent link="${name}_link" />
-      <child link="ardrone_base_${name}cam"/>
-    </joint>
-    <link name="ardrone_base_${name}cam">
-      <inertial>
-        <mass value="0.01" />
-        <origin xyz="0 0 0" />
-        <inertia ixx="0.001"  ixy="0.0"  ixz="0.0"
-                 iyy="0.001"  iyz="0.0"
-                 izz="0.001" />
-      </inertial>
-      <visual>
-        <origin xyz="0 0 0" rpy="0 0 0"/>
-        <geometry>
-          <box size="0.001 0.001 0.001" />
-        </geometry>
-      </visual>
-      <collision>
-        <origin xyz="0 0 0" rpy="0 0 0"/>
-        <geometry>
-          <box size="0.001 0.001 0.001" />
-        </geometry>
-      </collision>
-    </link>
-    <gazebo reference="${name}_link">
-      <sensor type="camera" name="${name}_camera_sensor">
-        <update_rate>${update_rate}</update_rate>
-        <camera name="head">
-          <horizontal_fov>${hfov}</horizontal_fov>
-          <image>
-            <width>${res_x}</width>
-            <height>${res_y}</height>
-            <format>${image_format}</format>
-          </image>
-          <clip>0.01
-	    <near>0.01</near>
-            <far>100</far>
-          </clip>
-        </camera>
-        <plugin name="${name}_camera_controller" filename="libgazebo_ros_camera.so">
-	  <cameraName>/${sim_name}/${name}</cameraName>
-          <alwaysOn>true</alwaysOn>
-          <updateRate>${update_rate}</updateRate>
-          <imageTopicName>/${sim_name}/${name}/image_raw</imageTopicName>
-          <cameraInfoTopicName>/${sim_name}/${name}/camera_info</cameraInfoTopicName>
-          <frameName>ardrone_base_${name}cam</frameName>
-        </plugin>
-      </sensor>
-      <turnGravityOff>true</turnGravityOff>
-      <material>PR2/Blue</material>
-    </gazebo>
-    </xacro:macro>
-  </robot>
+<robot xmlns:xacro="http://www.ros.org/wiki/xacro">
+<xacro:property name="M_PI" value="3.1415926535897931" />
+<xacro:macro name="generic_camera" params="name sim_name parent *origin update_rate res_x res_y image_format hfov">
+	<joint name="${name}_joint" type="fixed">
+		<xacro:insert_block name="origin" />
+    <parent link="${parent}"/>
+    <child link="${name}_link"/>
+  </joint>
+  <link name="${name}_link">
+		<visual>
+			<origin xyz="0 0 0" rpy="0 0 0" />
+			<geometry>
+				<box size="0.01 0.01 0.01" />
+			</geometry>
+			<material name="Blue">
+				<color rgba="0.0 0.0 0.8 1"/>
+			</material>
+		</visual>
+		<!--collision>
+			<origin xyz="0 0 0" rpy="0 0 0" />
+			<geometry>
+				<box size="0.01 0.01 0.01" />
+			</geometry>
+		</collision-->
+	</link>
+	<gazebo reference="${name}_link">
+		<sensor type="camera" name="${name}_camera_sensor">
+			<update_rate>${update_rate}</update_rate>
+			<camera name="head">
+				<horizontal_fov>${hfov}</horizontal_fov>
+				<image>
+					<width>${res_x}</width>
+					<height>${res_y}</height>
+					<format>${image_format}</format>
+				</image>
+				<clip>
+					<near>0.01</near>
+					<far>100</far>
+				</clip>
+			</camera>
+			<plugin name="${name}_camera_controller" filename="libgazebo_ros_camera.so">
+				<cameraName>/${sim_name}/${name}</cameraName>
+				<alwaysOn>true</alwaysOn>
+				<updateRate>${update_rate}</updateRate>
+				<imageTopicName>/${sim_name}/${name}/image_raw</imageTopicName>
+				<cameraInfoTopicName>/${sim_name}/${name}/camera_info</cameraInfoTopicName>
+				<frameName>ardrone_base_${name}cam</frameName>
+			</plugin>
+		</sensor>
+	</gazebo>
+</xacro:macro>
+</robot>

File: cvg_sim_gazebo/urdf/sensors/sonar_sensor.urdf.xacro (robot description, xacro)
@@ -1,63 +1,56 @@
 <?xml version="1.0"?>
-<robot xmlns:sensor="http://playerstage.sourceforge.net/gazebo/xmlschema/#sensor"
-xmlns:controller="http://playerstage.sourceforge.net/gazebo/xmlschema/#controller"
-xmlns:interface="http://playerstage.sourceforge.net/gazebo/xmlschema/#interface"
-xmlns:xacro="http://ros.org/wiki/xacro"
->
-  <xacro:macro name="sonar_sensor" params="name parent *origin ros_topic update_rate min_range max_range field_of_view ray_count">
-    <joint name="${name}_joint" type="fixed">
-      <xacro:insert_block name="origin" />
-      <parent link="${parent}"/>
-      <child link="${name}_link"/>
-    </joint>
-    <link name="${name}_link">
-      <inertial>
-        <mass value="0.001" />
-        <origin xyz="0 0 0" rpy="0 0 0" />
-        <inertia ixx="0.000000017" ixy="0" ixz="0" iyy="0.000000017" iyz="0" izz="0.000000017" />
-      </inertial>
-      <visual>
-        <origin xyz="0 0 0" rpy="0 0 0" />
-        <geometry>
-          <!--<box size="0.01 0.01 0.01" /> -->
-          <mesh filename="package://cvg_sim_gazebo/meshes/sonar_sensor/max_sonar_ez4.dae"/>
-        </geometry>
-      </visual>
-      <collision>
-        <origin xyz="0 0 0" rpy="0 0 0" />
-        <geometry>
-          <box size="0.01 0.01 0.01" />
-        </geometry>
-      </collision>
-    </link>
-    <gazebo reference="${name}_link">
-      <sensor type="ray" name="${name}">
-        <update_rate>${update_rate}</update_rate>
-        <ray>
-          <range>
-            <min>${min_range}</min>
-            <max>${max_range}</max>
-            <resolution>0.01</resolution>
-          </range>
-          <scan>
-            <horizontal>
-              <samples>${ray_count}</samples>
-              <min_angle>-${field_of_view/2}</min_angle>
-              <max_angle>${field_of_view/2}</max_angle>
-            </horizontal>
-            <vertical>
-              <samples>${ray_count}</samples>
-              <min_angle>-${field_of_view/2}</min_angle>
-              <max_angle>${field_of_view/2}</max_angle>
-            </vertical>
-          </scan>
-        </ray>
-        <plugin name="gazebo_ros_${name}_controller" filename="libhector_gazebo_ros_sonar.so">
-          <gaussianNoise>0.000</gaussianNoise>
-          <topicName>${ros_topic}</topicName>
-          <frameId>${name}_link</frameId>
-        </plugin>
-      </sensor>
-    </gazebo>
-  </xacro:macro>
+<robot xmlns:xacro="http://www.ros.org/wiki/xacro">
+<xacro:macro name="sonar_sensor" params="name parent *origin ros_topic update_rate min_range max_range field_of_view ray_count">
+	<joint name="${name}_joint" type="fixed">
+		<xacro:insert_block name="origin" />
+		<parent link="${parent}"/>
+		<child link="${name}_link"/>
+	</joint>
+	<link name="${name}_link">
+		<visual>
+			<origin xyz="0 0 0" rpy="0 0 0" />
+			<geometry>
+				<box size="0.01 0.01 0.01" />
+			</geometry>
+		</visual>
+		<!--collision>
+			<origin xyz="0 0 0" rpy="0 0 0" />
+			<geometry>
+				<box size="0.01 0.01 0.01" />
+			</geometry>
+		</collision-->
+	</link>
+	<gazebo reference="${name}_link">
+		<sensor type="ray" name="${name}">
+			<update_rate>${update_rate}</update_rate>
+			<ray>
+				<range>
+					<min>${min_range}</min>
+					<max>${max_range}</max>
+					<resolution>0.01</resolution>
+				</range>
+				<scan>
+					<horizontal>
+						<samples>${ray_count}</samples>
+						<min_angle>-${field_of_view/2}</min_angle>
+						<max_angle>${field_of_view/2}</max_angle>
+					</horizontal>
+					<vertical>
+						<samples>${ray_count}</samples>
+						<min_angle>-${field_of_view/2}</min_angle>
+						<max_angle>${field_of_view/2}</max_angle>
+					</vertical>
+				</scan>
+			</ray>
+			<plugin name="gazebo_ros_${name}_controller" filename="libhector_gazebo_ros_sonar.so">
+				<gaussianNoise>0.000</gaussianNoise>
+				<topicName>${ros_topic}</topicName>
+				<frameId>${name}_link</frameId>
+				<offset>0.0</offset>
+				<drift>0.0</drift>
+				<driftFrequency>0.0</driftFrequency>
+			</plugin>
+		</sensor>
+	</gazebo>
+</xacro:macro>
 </robot>

Commit message: robot namespace, so that we can spawn multiple drones at once

File: cvg_sim_gazebo/urdf/quadrotor.urdf.xacro (robot description, xacro)
@@ -26,9 +26,9 @@
 	</link>
 	<!-- Forward facing camera -->
-	<xacro:generic_camera name="front" sim_name="ardrone" parent="base_link" update_rate="60" res_x="640" res_y="360" image_format="R8G8B8" hfov="${81*M_PI/180}">
+	<xacro:generic_camera name="front" parent="base_link" update_rate="60" res_x="640" res_y="360" image_format="R8G8B8" hfov="${81*M_PI/180}">
 		<origin xyz="0.21 0.0 0.01" rpy="0 0 0"/>
 	</xacro:generic_camera>
 	<!-- Downward facing camera -->
-	<xacro:generic_camera name="bottom" sim_name="ardrone" parent="base_link" update_rate="60" res_x="640" res_y="360" image_format="R8G8B8" hfov="${81*M_PI/180}">
+	<xacro:generic_camera name="bottom" parent="base_link" update_rate="60" res_x="640" res_y="360" image_format="R8G8B8" hfov="${81*M_PI/180}">
 		<origin xyz="0.15 0.0 0.0" rpy="0 -${M_PI/2} 0"/>
 	</xacro:generic_camera>
@@ -46,5 +46,5 @@
         <bodyName>base_link</bodyName>
         <stateTopic>ground_truth/state</stateTopic>
-        <imuTopic>ardrone/imu</imuTopic>
+        <imuTopic>imu</imuTopic>
         <topicName>cmd_vel</topicName>
         <rollpitchProportionalGain>10.0</rollpitchProportionalGain>
@@ -70,5 +70,5 @@
         <bodyName>base_link</bodyName>
         <stateTopic>ground_truth/state</stateTopic>
-        <imuTopic>ardrone/imu</imuTopic>
+        <imuTopic>imu</imuTopic>
         <sonarTopic>sonar_height</sonarTopic>
         <topicName>cmd_vel</topicName>
@@ -79,5 +79,5 @@
 				<bodyName>base_link</bodyName>
 				<frameId>ardrone_base_link</frameId>
-				<topicName>/ardrone/imu</topicName>
+				<topicName>imu</topicName>
 				<rpyOffsets>0 0 0</rpyOffsets> <!-- deprecated -->
 				<gaussianNoise>0</gaussianNoise>  <!-- deprecated -->

File: cvg_sim_gazebo/urdf/sensors/generic_camera.urdf.xacro (robot description, xacro)
@@ -2,5 +2,5 @@
 <robot xmlns:xacro="http://www.ros.org/wiki/xacro">
 <xacro:property name="M_PI" value="3.1415926535897931" />
-<xacro:macro name="generic_camera" params="name sim_name parent *origin update_rate res_x res_y image_format hfov">
+<xacro:macro name="generic_camera" params="name parent *origin update_rate res_x res_y image_format hfov">
 	<joint name="${name}_joint" type="fixed">
 		<xacro:insert_block name="origin" />
@@ -41,9 +41,9 @@
 			</camera>
 			<plugin name="${name}_camera_controller" filename="libgazebo_ros_camera.so">
-				<cameraName>/${sim_name}/${name}</cameraName>
+				<cameraName>${name}</cameraName>
 				<alwaysOn>true</alwaysOn>
 				<updateRate>${update_rate}</updateRate>
-				<imageTopicName>/${sim_name}/${name}/image_raw</imageTopicName>
-				<cameraInfoTopicName>/${sim_name}/${name}/camera_info</cameraInfoTopicName>
+				<imageTopicName>${name}/image_raw</imageTopicName>
+				<cameraInfoTopicName>${name}/camera_info</cameraInfoTopicName>
 				<frameName>ardrone_base_${name}cam</frameName>
 			</plugin>

Commit message: fixed camera topics and camera bottom direction

File: cvg_sim_gazebo/urdf/quadrotor.urdf.xacro (robot description, xacro)
@@ -31,5 +31,5 @@
 	<!-- Downward facing camera -->
 	<xacro:generic_camera name="bottom" parent="base_link" update_rate="60" res_x="640" res_y="360" image_format="R8G8B8" hfov="${81*M_PI/180}">
-		<origin xyz="0.15 0.0 0.0" rpy="0 -${M_PI/2} 0"/>
+		<origin xyz="0.15 0.0 0.0" rpy="0 ${M_PI/2} 0"/>
 	</xacro:generic_camera>
 	<!-- Sonar height sensor -->

File: cvg_sim_gazebo/urdf/sensors/generic_camera.urdf.xacro (robot description, xacro)
@@ -44,6 +44,6 @@
 				<alwaysOn>true</alwaysOn>
 				<updateRate>${update_rate}</updateRate>
-				<imageTopicName>${name}/image_raw</imageTopicName>
-				<cameraInfoTopicName>${name}/camera_info</cameraInfoTopicName>
+				<imageTopicName>image_raw</imageTopicName>
+				<cameraInfoTopicName>camera_info</cameraInfoTopicName>
 				<frameName>ardrone_base_${name}cam</frameName>
 			</plugin>
